File: circuit/smith_corona.brd (EAGLE design)
At the start: 60.9 x 63.2 mm, 33 parts, among them Q1 2N3904, Q10 2N3904, Q11 2N3904, Q12 2N3904, Q13 2N3904, Q14 2N3904, Q15 2N3904, Q2 2N3904, Q3 2N3904, Q4 2N3904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

Commit message: tweak some wires
Parts:
- moved Q13 9.16 mm to (39.4, 12.7)
- moved Q14 9.16 mm to (39.4, 20.3)
- moved JP1 9.16 mm to (2.54, 48.3)
- moved JP2 9.16 mm to (43.2, 48.3)
- moved Q1 9.16 mm to (6.35, 12.7)
- moved Q4 9.16 mm to (11.4, 12.7)
- moved Q7 9.16 mm to (21.6, 12.7)
- moved Q11 9.16 mm to (34.3, 12.7)
- moved Q15 9.16 mm to (44.5, 12.7)
- moved Q2 9.16 mm to (6.35, 20.3)
- moved Q3 9.16 mm to (11.4, 20.3)
- moved Q6 9.16 mm to (16.5, 12.7)
- moved Q9 9.16 mm to (29.2, 12.7)
- moved R1 9.16 mm to (2.54, 36.8)
- moved R14 9.16 mm to (30.5, 36.8)
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Routing:
- net N$11: track 39.0 -> 33.8 mm
- net N$5: track 18.9 -> 16.7 mm
- net RIBBON14: track 23.9 -> 22.4 mm
- net RIBBON4: track 23.9 -> 23.2 mm
- net RIBBON11: track 10.2 -> 9.42 mm
- net RIBBON9: track 10.2 -> 9.42 mm
- net RIBBON2: track 23.9 -> 23.2 mm
Other:
- board size 60.9 x 63.2 mm -> 50.8 x 55.5 mm

Commit message: fix board more
Parts:
- flipped R10 to the top
- flipped R14 to the top
- flipped R15 to the top
- flipped R9 to the top
Routing:
- net N$11: track 33.8 -> 20.4 mm
- net N$3: track 18.9 -> 12.2 mm
- net N$15: track 27.1 -> 20.4 mm
- net N$13: track 27.1 -> 20.4 mm
- net RIBBON2: track 23.2 -> 17.1 mm
- net RIBBON4: track 23.2 -> 17.1 mm
- net RIBBON14: track 22.4 -> 17.1 mm
- net N$5: track 16.7 -> 12.2 mm
- net N$9: track 22.3 -> 20.4 mm
- net N$6: track 21.3 -> 19.6 mm
- net N$4: track 21.3 -> 19.6 mm
- net RIBBON10: track 18.1 -> 17.1 mm
- net RIBBON12: track 18.1 -> 17.1 mm
